Commit message: Update roboracer max vehicle description and launch files.

File: vehicle/roboracer_max_launch/roboracer_max_description/urdf/vehicle.xacro (robot description, xacro)
@@ -8,5 +8,5 @@
       <origin xyz="0 0 0" rpy="0 0 0"/>
       <geometry>
-        <mesh filename="package://roboracer_max_description/mesh/AV4EV_gokart.dae" scale="1 1 1"/>
+        <mesh filename="package://roboracer_max_description/mesh/roboracer_max.stl" scale="1 1 1"/>
       </geometry>
     </visual>
