Commit message: Tweaked sensor kit and vehicle definition on physical car

File: sensor_kit/roboracer_offroad_sensor_kit_launch/roboracer_offroad_sensor_kit_description/urdf/zed_macro.urdf.xacro (robot description, xacro)
@@ -205,9 +205,9 @@
         <parent link="${name}_camera_center"/>
         <child link="${name}_left_camera_frame"/>
-        <origin xyz="${optical_offset_x} ${baseline/2} 0" rpy="0 0 -${M_PI/2}" />
+        <origin xyz="${optical_offset_x} ${baseline/2} 0" rpy="0 0 0" />
       </joint>
       <link name="${name}_left_camera_frame_optical"/>
       <joint name="${name}_left_camera_joint_optical" type="fixed">
-        <origin xyz="0 0 0" rpy="-${M_PI/2} 0.0 0.0"/>
+        <origin xyz="0 0 0" rpy="-${M_PI/2} 0.0 -${M_PI/2}"/>
         <parent link="${name}_left_camera_frame"/>
         <child link="${name}_left_camera_frame_optical"/>
@@ -236,9 +236,9 @@
         <parent link="${name}_camera_center"/>
         <child link="${name}_right_camera_frame"/>
-        <origin xyz="${optical_offset_x} -${baseline/2} 0" rpy="0 0 -${M_PI/2}" />
+        <origin xyz="${optical_offset_x} -${baseline/2} 0" rpy="0 0 0" />
       </joint>
       <link name="${name}_right_camera_frame_optical"/>
       <joint name="${name}_right_camera_joint_optical" type="fixed">
-        <origin xyz="0 0 0" rpy="-${M_PI/2} 0.0 0"/>
+        <origin xyz="0 0 0" rpy="-${M_PI/2} 0.0 -${M_PI/2}"/>
         <parent link="${name}_right_camera_frame"/>
         <child link="${name}_right_camera_frame_optical"/>
